Commit message: GaryUpdateNavigation

File: meeting/src/robot_base/urdf/robot_base.urdf (robot description, URDF)
Before this commit: robot robot_base, 6 links, 5 joints
Links:
- removed link front_left_wheel
- removed link front_right_wheel
- removed link rear_left_wheel
- removed link rear_right_wheel
- added link base_footprint
- added link front_sensor; visual mesh filename=package://robot_base/meshes/urm04.STL scale=0.001 0.001 0.001
- added link left_sensor; visual mesh filename=package://robot_base/meshes/urm04.STL scale=0.001 0.001 0.001
- added link lower_left_wheel, mass 0.3844; collision cylinder length=0.0505 radius=0.05; visual mesh filename=package://robot_base/meshes/mecanum_wheel_right.STL scale=0.001 0.001 0.001
- added link lower_left_wheel_shaft, mass 0.055; collision mesh filename=package://robot_base/meshes/wheel_shaft.STL scale=0.001 0.001 0.001; visual mesh filename=package://robot_base/meshes/wheel_shaft.STL scale=0.001 0.001 0.001
- added link lower_right_wheel, mass 0.3844; collision cylinder length=0.0505 radius=0.05; visual mesh filename=package://robot_base/meshes/mecanum_wheel_left.STL scale=0.001 0.001 0.001
- added link lower_right_wheel_shaft, mass 0.055; collision mesh filename=package://robot_base/meshes/wheel_shaft.STL scale=0.001 0.001 0.001; visual mesh filename=package://robot_base/meshes/wheel_shaft.STL scale=0.001 0.001 0.001
- added link rear_sensor; visual mesh filename=package://robot_base/meshes/urm04.STL scale=0.001 0.001 0.001
- added link right_sensor; visual mesh filename=package://robot_base/meshes/urm04.STL scale=0.001 0.001 0.001
- added link upper_left_wheel, mass 0.3844; collision cylinder length=0.0505 radius=0.05; visual mesh filename=package://robot_base/meshes/mecanum_wheel_left.STL scale=0.001 0.001 0.001
- added link upper_left_wheel_shaft, mass 0.055; collision mesh filename=package://robot_base/meshes/wheel_shaft.STL scale=0.001 0.001 0.001; visual mesh filename=package://robot_base/meshes/wheel_shaft.STL scale=0.001 0.001 0.001
- added link upper_right_wheel, mass 0.3844; collision cylinder length=0.0505 radius=0.05; visual mesh filename=package://robot_base/meshes/mecanum_wheel_right.STL scale=0.001 0.001 0.001
- added link upper_right_wheel_shaft, mass 0.055; collision mesh filename=package://robot_base/meshes/wheel_shaft.STL scale=0.001 0.001 0.001; visual mesh filename=package://robot_base/meshes/wheel_shaft.STL scale=0.001 0.001 0.001
- link base_link: mass 0.70548109161444 -> 2.844; geometry collision mesh filename=package://robot_base/meshes/nexus_base_link_collision.STL scale=0.001 0.001 0.001; visual mesh filename=package://robot_base/meshes/nexus_base_link.STL scale=0.001 0.001 0.001
Joints:
- removed joint front_left_wheel_joint
- removed joint front_right_wheel_joint
- removed joint rear_left_wheel_joint
- removed joint rear_right_wheel_joint
- added joint base_link_joint: type fixed, parent base_footprint, child base_link, origin xyz=0 0 0.05 rpy=0 0 0
- added joint front_sensor_joint: type fixed, parent base_link, child front_sensor, origin xyz=0.205 0 0.010 rpy=0 0 0
- added joint left_sensor_joint: type fixed, parent base_link, child left_sensor, origin xyz=0 0.108 0.010 rpy=0 0 1.57079632679
- added joint lower_left_wheel_joint: type continuous, parent lower_left_wheel_shaft, child lower_left_wheel, origin xyz=0 0.042 0 rpy=0 0 0, axis 0 1 0
- added joint lower_left_wheel_shaft_joint: type fixed, parent base_link, child lower_left_wheel_shaft, origin xyz=-0.150 0.108 0.0 rpy=0 0 0
- added joint lower_right_wheel_joint: type continuous, parent lower_right_wheel_shaft, child lower_right_wheel, origin xyz=0 0.042 0 rpy=0 0 0, axis 0 1 0
- added joint lower_right_wheel_shaft_joint: type fixed, parent base_link, child lower_right_wheel_shaft, origin xyz=-0.150 -0.108 0.0 rpy=3.14159265359 0 0
- added joint rear_sensor_joint: type fixed, parent base_link, child rear_sensor, origin xyz=-0.201 0 0.010 rpy=0 0 3.14159265359
- added joint right_sensor_joint: type fixed, parent base_link, child right_sensor, origin xyz=0 -0.108 0.010 rpy=0 0 -1.57079632679
- added joint upper_left_wheel_joint: type continuous, parent upper_left_wheel_shaft, child upper_left_wheel, origin xyz=0 0.042 0 rpy=0 0 0, axis 0 1 0
- added joint upper_left_wheel_shaft_joint: type fixed, parent base_link, child upper_left_wheel_shaft, origin xyz=0.150 0.108 0.0 rpy=0 0 0
- added joint upper_right_wheel_joint: type continuous, parent upper_right_wheel_shaft, child upper_right_wheel, origin xyz=0 0.042 0 rpy=0 0 0, axis 0 1 0
- added joint upper_right_wheel_shaft_joint: type fixed, parent base_link, child upper_right_wheel_shaft, origin xyz=0.150 -0.108 0.0 rpy=3.14159265359 0 0

Commit message: k

File: meeting/src/robot_base/urdf/robot_base.urdf (robot description, URDF)
Before this commit: robot robot_base, 15 links, 14 joints
Links:
- added link cameraLeft_depth_link
- added link kinect_camera_link, mass 0.1; collision box size=0.073000 0.276000 0.072000; visual mesh filename=/home/flynn/.gazebo/models/kinect/meshes/kinect.dae
Joints:
- added joint cameraLeft_depth_joint: type fixed, parent kinect_camera_link, child cameraLeft_depth_link, origin xyz=0 0 0 rpy=-1.5708 0 -1.5708 
- added joint kinect_camera_joint: type fixed, parent base_link, child kinect_camera_link, origin xyz=0 0 0.3 rpy=0 0 0

Commit message: small change

File: meeting/src/robot_base/urdf/robot_base.urdf (robot description, URDF)
Before this commit: robot robot_base, 17 links, 16 joints
Links:
- removed link cameraLeft_depth_link
- removed link kinect_camera_link
- removed link laser_link
- added link camera_link, mass 0.1; collision box size=0.073000 0.276000 0.072000; visual mesh filename=/home/flynn/.gazebo/models/kinect/meshes/kinect.dae
- added link laser; visual cylinder length=0.02 radius=0.05
Joints:
- removed joint base_laser_joint
- removed joint cameraLeft_depth_joint
- added joint laser: type fixed, parent base_link, child laser, origin xyz=0.290 0.0 0.640 rpy=0 0 0
- joint base_link_joint: origin xyz=0 0 0.05 rpy=0 0 0 -> xyz=0 0 0.07 rpy=0 0 0
- joint front_sensor_joint: origin xyz=0.205 0 0.010 rpy=0 0 0 -> xyz=0.39 0 0.0 rpy=0 0 0
- joint kinect_camera_joint: child kinect_camera_link -> camera_link; origin xyz=0 0 0.3 rpy=0 0 0 -> xyz=0.27 0 0.1 rpy=0 0 0
- joint left_sensor_joint: origin xyz=0 0.108 0.010 rpy=0 0 1.57079632679 -> xyz=0 0.175 -0.025 rpy=0 0 1.57079632679
- joint lower_left_wheel_shaft_joint: origin xyz=-0.150 0.108 0.0 rpy=0 0 0 -> xyz=-0.145 0.17 -0.115 rpy=0 0 0
- joint lower_right_wheel_shaft_joint: origin xyz=-0.150 -0.108 0.0 rpy=3.14159265359 0 0 -> xyz=-0.145 -0.17 -0.115 rpy=3.14159265359 0 0
- joint rear_sensor_joint: origin xyz=-0.201 0 0.010 rpy=0 0 3.14159265359 -> xyz=-0.22 0 -0.025 rpy=0 0 3.14159265359
- joint right_sensor_joint: origin xyz=0 -0.108 0.010 rpy=0 0 -1.57079632679 -> xyz=0 -0.175 -0.025 rpy=0 0 -1.57079632679
- joint upper_left_wheel_shaft_joint: origin xyz=0.150 0.108 0.0 rpy=0 0 0 -> xyz=0.20 0.17 -0.115 rpy=0 0 0
- joint upper_right_wheel_shaft_joint: origin xyz=0.150 -0.108 0.0 rpy=3.14159265359 0 0 -> xyz=0.20 -0.17 -0.115 rpy=3.14159265359 0 0

Commit message: working code

File: meeting/src/robot_base/urdf/robot_base.urdf (robot description, URDF)
Before this commit: robot robot_base, 16 links, 15 joints
Joints:
- joint laser: origin xyz=0.290 0.0 0.640 rpy=0 0 0 -> xyz=0.290 0.0 0.640 rpy=0 0 3.14
